File: pcb/sdcard.kicad_sch (KiCad schematic)
At the start: 10 parts, among them J4 Micro_SD_Card_Det1

Commit message: fix: add FET to measurement circuit
Disable the battery measurement circuit when the device is switched off to save energy
Parts:
- renumbered C2 to C4, C3 to C5, R1 to R7, R2 to R8
Changed lines of the file:
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@@
 		(on_board yes)
 		(dnp no)
-		(property "Reference" "#PWR030"
+		(property "Reference" "#PWR036"
 			(at 194.31 109.22 0)
 			(effects
@@
 			(project "Badge-Scanner"
 				(path "/e99cd76d-c117-4654-ad48-596a9e3de149/265dd7b3-4c57-4927-af43-2ab583aa098f"
-					(reference "#PWR030")
+					(reference "#PWR036")
 					(unit 1)
 				)
@@
 		(on_board yes)
 		(dnp no)
-		(property "Reference" "#PWR029"
+		(property "Reference" "#PWR035"
 			(at 146.05 109.22 0)
 			(effects
@@
 			(project "Badge-Scanner"
 				(path "/e99cd76d-c117-4654-ad48-596a9e3de149/265dd7b3-4c57-4927-af43-2ab583aa098f"
-					(reference "#PWR029")
+					(reference "#PWR035")
 					(unit 1)
 				)
@@
 		(on_board yes)
 		(dnp no)
-		(property "Reference" "#PWR015"
+		(property "Reference" "#PWR033"
 			(at 160.02 53.34 0)
 			(effects
@@
 			(project "Badge-Scanner"
 				(path "/e99cd76d-c117-4654-ad48-596a9e3de149/265dd7b3-4c57-4927-af43-2ab583aa098f"
-					(reference "#PWR015")
+					(reference "#PWR033")
 					(unit 1)
 				)
@@
 		(dnp no)
 		(fields_autoplaced yes)
-		(property "Reference" "#PWR09"
+		(property "Reference" "#PWR032"
 			(at 146.05 52.07 0)
 			(effects
@@
 			(project "Badge-Scanner"
 				(path "/e99cd76d-c117-4654-ad48-596a9e3de149/265dd7b3-4c57-4927-af43-2ab583aa098f"
-					(reference "#PWR09")
+					(reference "#PWR032")
 					(unit 1)
 				)
@@
 		(dnp no)
 		(fields_autoplaced yes)
-		(property "Reference" "C3"
+		(property "Reference" "C5"
 			(at 151.1237 56.5236 90)
 			(effects
@@
 			(project "Badge-Scanner"
 				(path "/e99cd76d-c117-4654-ad48-596a9e3de149/265dd7b3-4c57-4927-af43-2ab583aa098f"
-					(reference "C3")
+					(reference "C5")
 					(unit 1)
 				)
@@
 		(on_board yes)
 		(dnp no)
-		(property "Reference" "R1"
+		(property "Reference" "R7"
 			(at 124.2314 67.3679 0)
 			(effects
@@
 			(project "Badge-Scanner"
 				(path "/e99cd76d-c117-4654-ad48-596a9e3de149/265dd7b3-4c57-4927-af43-2ab583aa098f"
-					(reference "R1")
+					(reference "R7")
 					(unit 1)
 				)
@@
 		(dnp no)
 		(fields_autoplaced yes)
-		(property "Reference" "C2"
+		(property "Reference" "C4"
 			(at 151.1236 46.99 90)
 			(effects
@@
 			(project "Badge-Scanner"
 				(path "/e99cd76d-c117-4654-ad48-596a9e3de149/265dd7b3-4c57-4927-af43-2ab583aa098f"
-					(reference "C2")
+					(reference "C4")
 					(unit 1)
 				)
@@
 		(on_board yes)
 		(dnp no)
-		(property "Reference" "#PWR019"
+		(property "Reference" "#PWR034"
 			(at 160.02 62.23 0)
 			(effects
@@
 			(project "Badge-Scanner"
 				(path "/e99cd76d-c117-4654-ad48-596a9e3de149/265dd7b3-4c57-4927-af43-2ab583aa098f"
-					(reference "#PWR019")
+					(reference "#PWR034")
 					(unit 1)
 				)
@@
 		(dnp no)
 		(fields_autoplaced yes)
-		(property "Reference" "R2"
+		(property "Reference" "R8"
 			(at 129.7686 67.3679 0)
 			(effects
@@
 			(project "Badge-Scanner"
 				(path "/e99cd76d-c117-4654-ad48-596a9e3de149/265dd7b3-4c57-4927-af43-2ab583aa098f"
-					(reference "R2")
-					(unit 1)
-				)
+					(reference "R8")
+					(unit 1)
+				)
