File: pcb/battery.kicad_sch (KiCad schematic)
At the start: 26 parts, among them Q2 AO3401A, Q3 AO3401A, Q5 AO3400A, Q6 AO3400A, Q7 AO3401A, Q8 AO3400A, SW1 Power, U3 TP4056

Commit message: feat: add reset button
Parts:
- added SW2: Reset, Button_Switch_THT:SW_Tactile_SPST_Angled_PTS645Vx31-2LFS, symbol Switch:SW_Push
Connections:
- net BattSw: now also SW2.1
- net GND: now also SW2.2
Changed lines of the file:
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@@
+	(wire
+		(pts
+			(xy 173.99 71.12) (xy 177.8 71.12)
+		)
+		(stroke
+			(width 0)
+			(type default)
+		)
+	)
 	(wire
 		(pts
@@
 	(wire
 		(pts
+			(xy 157.48 71.12) (xy 163.83 71.12)
+		)
+		(stroke
+			(width 0)
+			(type default)
+		)
+	)
+	(wire
+		(pts
 			(xy 50.8 73.66) (xy 50.8 76.2)
 		)
@@
 		(pts
 			(xy 142.24 87.63) (xy 142.24 90.17)
+		)
+		(stroke
+			(width 0)
+			(type default)
+		)
+	)
+	(wire
+		(pts
+			(xy 177.8 71.12) (xy 177.8 73.66)
 		)
 		(stroke
@@
 	)
 	(symbol
+		(lib_id "power:GND")
+		(at 177.8 73.66 0)
+		(unit 1)
+		(exclude_from_sim no)
+		(in_bom yes)
+		(on_board yes)
+		(dnp no)
+		(fields_autoplaced yes)
+		(property "Reference" "#PWR054"
+			(at 177.8 80.01 0)
+			(effects
+				(font
+					(size 1.27 1.27)
+				)
+				(hide yes)
+			)
+		)
+		(property "Value" "GND"
+			(at 177.8 78.74 0)
+			(effects
+				(font
+					(size 1.27 1.27)
+				)
+			)
+		)
+		(property "Footprint" ""
+			(at 177.8 73.66 0)
+			(effects
+				(font
+					(size 1.27 1.27)
+				)
+				(hide yes)
+			)
+		)
+		(property "Datasheet" ""
+			(at 177.8 73.66 0)
+			(effects
+				(font
+					(size 1.27 1.27)
+				)
+				(hide yes)
+			)
+		)
+		(property "Description" "Power symbol creates a global label with name \"GND\" , ground"
+			(at 177.8 73.66 0)
+			(effects
+				(font
+					(size 1.27 1.27)
+				)
+				(hide yes)
+			)
+		)
+		(pin "1"
+		)
+		(instances
+			(project "Badge-Scanner"
+				(path "/e99cd76d-c117-4654-ad48-596a9e3de149/0a7a7e59-ee25-477c-a5be-167264b2ebb9"
+					(reference "#PWR054")
+					(unit 1)
+				)
+			)
+		)
+	)
+	(symbol
 		(lib_id "Device:D_Schottky_Small")
 		(at 243.84 44.45 180)
@@
 					(unit 1)
 				)
+			)
+		)
+	)
+	(symbol
+		(lib_id "Switch:SW_Push")
+		(at 168.91 71.12 0)
+		(unit 1)
+		(exclude_from_sim no)
+		(in_bom yes)
+		(on_board yes)
+		(dnp no)
+		(fields_autoplaced yes)
+		(property "Reference" "SW2"
+			(at 168.91 63.5 0)
+			(effects
+				(font
+					(size 1.27 1.27)
+				)
+			)
+		)
+		(property "Value" "Reset"
+			(at 168.91 66.04 0)
+			(effects
+				(font
+					(size 1.27 1.27)
+				)
+			)
+		)
+		(property "Footprint" "Button_Switch_THT:SW_Tactile_SPST_Angled_PTS645Vx31-2LFS"
+			(at 168.91 66.04 0)
+			(effects
+				(font
+					(size 1.27 1.27)
+				)
+				(hide yes)
+			)
+		)
+		(property "Datasheet" "~"
+			(at 168.91 66.04 0)
+			(effects
+				(font
+					(size 1.27 1.27)
+				)
+				(hide yes)
+			)
+		)
+		(property "Description" "Push button switch, generic, two pins"
+			(at 168.91 71.12 0)
+			(effects
+				(font
+					(size 1.27 1.27)
+				)
+				(hide yes)
+			)
+		)
+		(pin "2"
+		)
+		(pin "1"
+		)
+		(instances
+			(project ""
+				(path "/e99cd76d-c117-4654-ad48-596a9e3de149/0a7a7e59-ee25-477c-a5be-167264b2ebb9"
+					(reference "SW2")
+					(unit 1)
+				)

Commit message: fix: re-release because of CI error
Other:
- note added: "Manual Power off override"
- moved on the sheet: SW2
Changed lines of the file:
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@@
 	(wire
 		(pts
-			(xy 173.99 71.12) (xy 177.8 71.12)
+			(xy 177.8 71.12) (xy 181.61 71.12)
 		)
 		(stroke
@@
 	(wire
 		(pts
-			(xy 157.48 71.12) (xy 163.83 71.12)
+			(xy 157.48 71.12) (xy 167.64 71.12)
 		)
 		(stroke
@@
 	(wire
 		(pts
-			(xy 177.8 71.12) (xy 177.8 73.66)
+			(xy 181.61 71.12) (xy 181.61 73.66)
 		)
 		(stroke
@@
 			(width 0)
 			(type default)
+		)
+	)
+	(rectangle
+		(start 166.37 58.42)
+		(end 195.58 82.55)
+		(stroke
+			(width 0)
+			(type dot)
+		)
+		(fill
+			(type none)
 		)
 	)
@@
 		(exclude_from_sim no)
 		(at 211.328 61.468 0)
+		(effects
+			(font
+				(size 1.27 1.27)
+			)
+		)
+	)
+	(text "Manual Power off override"
+		(exclude_from_sim no)
+		(at 180.848 61.214 0)
 		(effects
 			(font
@@
 	(symbol
 		(lib_id "power:GND")
-		(at 177.8 73.66 0)
+		(at 181.61 73.66 0)
 		(unit 1)
 		(exclude_from_sim no)
@@
 		(fields_autoplaced yes)
 		(property "Reference" "#PWR054"
-			(at 177.8 80.01 0)
+			(at 181.61 80.01 0)
 			(effects
 				(font
@@
 		)
 		(property "Value" "GND"
-			(at 177.8 78.74 0)
+			(at 181.61 78.74 0)
 			(effects
 				(font
@@
 		)
 		(property "Footprint" ""
-			(at 177.8 73.66 0)
+			(at 181.61 73.66 0)
 			(effects
 				(font
@@
 		)
 		(property "Datasheet" ""
-			(at 177.8 73.66 0)
+			(at 181.61 73.66 0)
 			(effects
 				(font
@@
 		)
 		(property "Description" "Power symbol creates a global label with name \"GND\" , ground"
-			(at 177.8 73.66 0)
+			(at 181.61 73.66 0)
 			(effects
 				(font
@@
 	(symbol
 		(lib_id "Switch:SW_Push")
-		(at 168.91 71.12 0)
+		(at 172.72 71.12 0)
 		(unit 1)
 		(exclude_from_sim no)
@@
 		(fields_autoplaced yes)
 		(property "Reference" "SW2"
-			(at 168.91 63.5 0)
+			(at 172.72 63.5 0)
 			(effects
 				(font
@@
 		)
 		(property "Value" "Reset"
-			(at 168.91 66.04 0)
+			(at 172.72 66.04 0)
 			(effects
 				(font
@@
 		)
 		(property "Footprint" "Button_Switch_THT:SW_Tactile_SPST_Angled_PTS645Vx31-2LFS"
-			(at 168.91 66.04 0)
+			(at 172.72 66.04 0)
 			(effects
 				(font
@@
 		)
 		(property "Datasheet" "~"
-			(at 168.91 66.04 0)
+			(at 172.72 66.04 0)
 			(effects
 				(font
@@
 		)
 		(property "Description" "Push button switch, generic, two pins"
-			(at 168.91 71.12 0)
-			(effects
-				(font
+			(at 172.72 71.12 0)
+			(effects
+				(font
